Commit message: Kobuki: spherical wheel collisions
A cylinder's contact with the floor jumps between its rims, so odometry
drifted ~8 % when spinning in place. A sphere of the same radius keeps
the contact on the wheel's mid plane.

Fixes #25

Signed-off-by: Francisco Martín Rico <fmrico@gmail.com>

File: playground_kobuki/easynav_playground_kobuki_description/urdf/kobuki_base.urdf.xacro (robot description, xacro)
@@ -68,7 +68,9 @@
         <origin xyz="0 0 0" rpy="0 0 0"/>
       </visual>
-      <collision>
-        <geometry>
-          <cylinder length="0.0206" radius="0.035"/>
+      <!-- A sphere touches the floor on the wheel's mid plane: a cylinder's contact
+           jumps between its rims and odometry drifts (8 % when spinning in place). -->
+      <collision>
+        <geometry>
+          <sphere radius="0.035"/>
         </geometry>
         <origin rpy="0 0 0" xyz="0 0 0"/>
@@ -95,7 +97,9 @@
         <origin xyz="0 0 0" rpy="0 0 0"/>
       </visual>
-      <collision>
-        <geometry>
-          <cylinder length="0.0206" radius="0.035"/>
+      <!-- A sphere touches the floor on the wheel's mid plane: a cylinder's contact
+           jumps between its rims and odometry drifts (8 % when spinning in place). -->
+      <collision>
+        <geometry>
+          <sphere radius="0.035"/>
         </geometry>
         <origin rpy="0 0 0" xyz="0 0 0"/>
