Commit message: Kobuki: optional lidar target
A visual-only cylinder at the height of the lidar, so that other robots'
lidars see the robot. It lies inside the lidar's minimum range, where
gpu_lidar renders nothing: the robot's own scans do not change.

Fixes #27

Signed-off-by: Francisco Martín Rico <fmrico@gmail.com>

File: playground_kobuki/easynav_playground_kobuki_description/urdf/kobuki.urdf.xacro (robot description, xacro)
@@ -10,4 +10,8 @@
   <xacro:arg name="structure" default="false" />
   <xacro:arg name="lidar_range" default="12.0" />
+  <!-- A cylinder at the height of the lidar that other robots' lidars see (a Kobuki alone shows
+       them only its thin standoffs). Visual only, and inside the lidar's min range (0.17 m),
+       where its own lidar renders nothing: it does not hide anything from its own scans. -->
+  <xacro:arg name="lidar_target" default="false" />
   <!-- Namespace will be applied to all TF frames and topics.
        This is required if multiple robots are launched at the same time.
@@ -48,4 +52,21 @@
     <xacro:include filename="$(find easynav_playground_kobuki_description)/urdf/sensors/lidar.urdf.xacro"/>
     <xacro:sensor_lidar namespace="$(arg namespace)"/>
+    <xacro:if value="$(arg lidar_target)">
+      <link name="$(arg namespace)lidar_target_link">
+        <visual>
+          <geometry>
+            <cylinder length="0.10" radius="0.15"/>
+          </geometry>
+          <material name="lidar_target_orange">
+            <color rgba="1.0 0.5 0.0 1.0"/>
+          </material>
+        </visual>
+      </link>
+      <joint name="$(arg namespace)lidar_target_joint" type="fixed">
+        <origin xyz="0.0 0.0 0.0" rpy="0 0 0"/>
+        <parent link="$(arg namespace)laser_link"/>
+        <child link="$(arg namespace)lidar_target_link"/>
+      </joint>
+    </xacro:if>
   </xacro:if>
   <xacro:if value="$(arg camera)">
